File: TestingComp/RocketIgniter300/RocketIgniter300.sch (KiCad schematic (older format))
At the start: 12 parts

Commit message: Updated schematic
Signed-off-by: vaan3225 <63621952+Raggii@users.noreply.github.com>
Parts:
- removed U? (x5): 74LS125, symbol 74xx:74LS125
- removed U?: STM32F103CBTx, Package_QFP:LQFP-48_7x7mm_P0.5mm, symbol MCU_ST_STM32F1:STM32F103CBTx
- added 22pF1, 22pF2: C, symbol Device:C
- added 25MHz1: Crystal, symbol Device:Crystal
- added R1: 12k, symbol Device:R
- added R2: 20k, symbol Device:R
- added U4: 74AUC2G125, symbol 74xGxx:74AUC2G125
- added U5: STM32L053R8Tx, Package_QFP:LQFP-64_10x10mm_P0.5mm, symbol MCU_ST_STM32L0:STM32L053R8Tx
- gave numbers to parts that had none: 3
- renumbered j to j1, terminatingResistor to terminatingResistor1
Connections:
- net labels added: ClockPin1, ClockPin2, UartEnable2, VCC, VoltageMeasure
- wire segments 12 -> 23
Other:
- note added: "- Need a Voltage regulator!\n- Also need another way to get to 5V for the can line\n- Will the 5V break the microcontroller?"
- note added: "Can bus line with multiplexer\n- Has Tri State Buffers to convert between Uart and CanBus"
- note added: "Crystal Oscillator"
- note added: "Just some screw pins tbh\n- Do we need 1 or 2 tho?\n- just one"
- note added: "Voltage Measuring"
- note removed: "Extra TriStates if needed"
- note removed: "Might get the Nucleo stm32f103"
- moved on the sheet: U2, terminatingResistor1, terminatingResistor2
