File: CanNode/CanNode.kicad_pcb (KiCad board)
At the start: 2 copper layers, 19 parts, among them J1 Input Lipo, J2 IgnitOnePinOut, J3 InputCanBus, J4 IgnitTwoPinOut, Q1 AO4576, Q2 AO4576, U1 MCP2515-xSO, U2 MCP2551-I-P, U3 74AHC1G126, U4 74LS157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

Commit message: Updated the schematic somre more
Hope u can get it finished tomorrow!!
Parts:
- Q1, Q2: footprint Package_TO_SOT_SMD:LFPAK33 -> Package_TO_SOT_SMD:SOT-23-8_Handsoldering
- moved J3 201.3 mm to (53.3, 106.7), turned to 0 degrees
- moved U4 194.9 mm to (57.1, 74.3), turned to 0 degrees
- moved R2 176.6 mm to (53.3, 100.3), turned to 0 degrees
- moved U3 167.9 mm to (59.7, 106.7)
- moved R1 160.9 mm to (92.7, 95.2), turned to 90 degrees
- moved U5 156.6 mm to (80.0, 61.0), turned to 0 degrees
- moved U2 147.8 mm to (88.9, 105.4), turned to 270 degrees
- moved C3 144.7 mm to (72.4, 83.8), turned to 180 degrees
- moved U1 142.6 mm to (106.7, 94.0), turned to 180 degrees
- moved C4 142.2 mm to (72.4, 95.2), turned to 180 degrees
- moved Crystal2 141.9 mm to (74.9, 87.6), turned to 270 degrees
- moved C2 133.7 mm to (114.3, 71.1), turned to 0 degrees
- moved Crystal1 126.0 mm to (111.8, 78.7), turned to 90 degrees
- moved C1 121.4 mm to (114.3, 82.5)
- moved Q2 116.1 mm to (101.5, 105.4), turned to 180 degrees
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Routing:
- net GND: track 0.00 -> 84.3 mm
- net 5V: track 0.00 -> 62.0 mm
- net Rx: track 0.00 -> 31.1 mm
- net EnableUart: track 0.00 -> 25.2 mm
- net LipoBattery: track 0.00 -> 20.0 mm
- net ClockIn2: track 0.00 -> 14.6 mm
- net ClockIn1: track 0.00 -> 13.5 mm
- net Net-(C2-Pad1): track 0.00 -> 10.5 mm
- net Net-(C1-Pad1): track 0.00 -> 9.94 mm
Other:
- net class 5V added: clearance 0.2, trace_width 0.5, via_dia 0.8, via_drill 0.4
- net class HighCurrent added: clearance 0.2, trace_width 0.6, via_dia 0.8, via_drill 0.4
