File: CanNode/CanNode.sch (KiCad schematic (older format))
At the start: 19 parts

Commit message: Updated the foot prints
Added notes also
Parts:
- U3: renamed from U?; footprint (none) -> Libs:SOT65P210X110-5N
- gave numbers to parts that had none: 17
- renumbered Crystal to Crystal1
Connections:
- net CS: now also U5.17 (PB3)
- net ClockIn1: no longer U5.10 (XTAL2/PB7)
- net ClockIn2: now also U5.10 (XTAL2/PB7)
- net SCK: now also U5.16 (PB2)
- net SI: now also U5.19 (PB5)
- net SO: now also U5.18 (PB4)
Other:
- note added: "Also \n- Need to get foot print for the mosfet!"

Commit message: Updated the schematic somre more
Hope u can get it finished tomorrow!!
Parts:
- Q1, Q2: footprint Package_TO_SOT_SMD:LFPAK33 -> Package_TO_SOT_SMD:SOT-23-8_Handsoldering
Changed lines of the file:
@@
 F 0 "Q2" V 5149 5050 50  0000 C CNN
 F 1 "AO4576" V 5240 5050 50  0000 C CNN
-F 2 "Package_TO_SOT_SMD:LFPAK33" H 5100 4975 50  0001 L CIN
+F 2 "Package_TO_SOT_SMD:SOT-23-8_Handsoldering" H 5100 4975 50  0001 L CIN
 F 3 "https://assets.nexperia.com/documents/data-sheet/BUK7M42-60E.pdf" V 4900 5050 50  0001 L CNN
 	1    4900 5050
@@
 F 0 "Q1" V 3399 5050 50  0000 C CNN
 F 1 "AO4576" V 3490 5050 50  0000 C CNN
-F 2 "Package_TO_SOT_SMD:LFPAK33" H 3350 4975 50  0001 L CIN
+F 2 "Package_TO_SOT_SMD:SOT-23-8_Handsoldering" H 3350 4975 50  0001 L CIN
 F 3 "https://assets.nexperia.com/documents/data-sheet/BUK7M42-60E.pdf" V 3150 5050 50  0001 L CNN
 	1    3150 5050
